File: hw/shield-pcb/dynamics-accservo-shield/dynamics-accservo-shield.kicad_pcb (KiCad board)
At the start: 2 copper layers, 41.5 x 39.5 mm, 13 parts, among them J2 uStepperS32-shield, M2 Servo, U2 L7806

Commit message: added PCB design
Parts:
- removed EC1: 100u, Capacitor_SMD:CP_Elec_10x10
- added EC3: 220u, Capacitor_SMD:CP_Elec_6.3x7.7, F.Cu at (178.7, 61.2)
- added G***: LOGO, 000_Graphics_Immo:practactable.io_text_30x11, F.Cu at (147.8, 65.0)
- added G***: LOGO, 000_Graphics_Immo:Remote Labs SN Block, B.Cu at (153.4, 80.7)
- added G***: LOGO, 000_Graphics_Immo:practactable.io_text_80x30, B.Cu at (179.8, 71.4)
- added J3: MPU6050-module, 000_Modules_Immo:MPU6050-acc-module, F.Cu at (169.1, 57.2)
- D1: value LED_0805_Yellow -> 12v
- D2: value LED_0805_Blue -> 6v
- D3: value LED_0805_red -> beacon
- D4: value LED-TH -> beacon
- moved R2 50.9 mm to (183.5, 88.6), turned to 90 degrees
- moved R1 48.0 mm to (180.0, 88.6), turned to -90 degrees
- moved EC2 32.6 mm to (150.0, 88.5)
- moved R4 22.4 mm to (152.0, 75.0), turned to 90 degrees
- moved R3 19.1 mm to (152.0, 81.0), turned to 90 degrees
- moved D1 18.3 mm to (180.0, 82.3), turned to 90 degrees
- moved D2 15.8 mm to (183.5, 82.3), turned to 90 degrees
- moved D3 13.4 mm to (147.5, 81.0), turned to 90 degrees
- moved M2 12.5 mm to (182.0, 71.0)
- moved U2 7.39 mm to (165.8, 87.6)
- moved D4 2.30 mm to (146.5, 73.5), turned to -90 degrees
Connections:
- J2 pad 15: unconnected-(J2-D4-Pad15) -> /BEACON_LIGHT
- J2 pad 17: unconnected-(J2-D6-Pad17) -> /SERVO_PPM
- J2 pad 18: unconnected-(J2-D7-Pad18) -> /SCL
- J2 pad 19: unconnected-(J2-D8-Pad19) -> /SDA
- J2 pad 3: unconnected-(J2-5v-Pad3) -> /5V
Routing:
- net /12V_VIN: track 0.00 -> 57.2 mm, vias 0 -> 2
- net GND: track 0.00 -> 56.8 mm, vias 0 -> 2
- net /6V_SERVO: track 0.00 -> 55.4 mm
- net /BEACON_LIGHT: track 0.00 -> 47.3 mm
- net /SDA: track 0.00 -> 24.7 mm
- net /SCL: track 0.00 -> 24.1 mm, vias 0 -> 2
- net /5V: track 0.00 -> 23.7 mm
- net /SERVO_PPM: track 0.00 -> 9.58 mm
- net Net-(D4-K): track 0.00 -> 5.71 mm
- net Net-(D3-K): track 0.00 -> 5.33 mm
- net Net-(D2-K): track 0.00 -> 4.30 mm
- net Net-(D1-K): track 0.00 -> 4.30 mm
- added copper zone on B.Cu, net GND
- added copper zone on F.Cu, net GND

Commit message: finished hardware dev
Parts:
- removed EC3: 220u, Capacitor_SMD:CP_Elec_6.3x7.7
- added EC1: 1000uF, Capacitor_THT:CP_Radial_D13.0mm_P5.00mm, F.Cu at (180.4, 61.8)
Routing:
- net GND: track 56.8 -> 49.6 mm, vias 2 -> 1
- net /SDA: track 24.7 -> 22.2 mm
Other:
- board text added: "Design:"
- board text added: "Dynamics-Lab"
- board text added: "Imogen Heard"
- board text added: "uStepperS32 Shield V1.0"
