File: hw/shield-pcb/dynamics-accservo-shield/dynamics-accservo-shield.kicad_sch (KiCad schematic)
At the start: 13 parts, among them J2 uStepperS32-shield, M2 Servo, U2 L7806

Commit message: added PCB design
Parts:
- removed EC1: 100u, Capacitor_SMD:CP_Elec_10x10, symbol 000_Capacitor_Electrolytic_Immo:100u
- added EC3: 220u, Capacitor_SMD:CP_Elec_6.3x7.7, symbol 000_Capacitor_Electrolytic_Immo:220u
- added J3: MPU6050-module, 000_Modules_Immo:MPU6050-acc-module, symbol 000_Modules_Immo:MPU6050-accellerometer-module
- D1: value LED_0805_Yellow -> 12v
- D2: value LED_0805_Blue -> 6v
- D3: value LED_0805_red -> beacon
- D4: value LED-TH -> beacon
Connections:
- net 6V_SERVO: now also EC3.1
- net BEACON_LIGHT: now also J2.15 (D4)
- net GND: now also EC3.2, J3.2 (GND)
- net SERVO_PPM: now also J2.17 (D6)
- net SCL: now reaches J2.18 (D7)
- net SCL: now also J3.3 (SCL)
- net SDA: now reaches J2.19 (D8)
- net SDA: now also J3.4 (SDA)
- net 5V: now reaches J2.3 (5v)
- net 5V: now also J3.1 (Vcc)
- no-connect marks 0 -> 4
Other:
- moved on the sheet: J2, M2

Commit message: finished hardware dev
Parts:
- removed EC3: 220u, Capacitor_SMD:CP_Elec_6.3x7.7, symbol 000_Capacitor_Electrolytic_Immo:220u
- added EC1: 1000uF, Capacitor_THT:CP_Radial_D13.0mm_P5.00mm, symbol 000_Capacitor_Electrolytic_Immo:1000uF
- EC2: JLCpart C4747974 -> C3342
Connections:
- net 6V_SERVO: now also EC1.1
- net GND: now also EC1.2
Other:
- moved on the sheet: D2, R2
